Commit message: link pos chg & gazebo

File: urdf/iiwa_agv.gazebo.xacro (robot description, xacro)
@@ -3,66 +3,40 @@
   <gazebo reference="${prefix}agv_link">
     <material>Gazebo/Blue</material>
-    <mu1>0.5</mu1>
-    <mu2>0.5</mu2>
   </gazebo>
   <gazebo reference="${prefix}base_link">
     <material>Gazebo/Purple</material>
-    <mu1>0.5</mu1>
-    <mu2>0.5</mu2>
   </gazebo>
   <gazebo reference="${prefix}link_1">
       <material>Gazebo/Yellow</material>
-      <mu1>0.5</mu1>
-      <mu2>0.5</mu2>
   </gazebo>
   <gazebo reference="${prefix}link_2">
       <material>Gazebo/Red</material>
-      <mu1>0.5</mu1>
-      <mu2>0.5</mu2>
   </gazebo>
   <gazebo reference="${prefix}link_3">
       <material>Gazebo/Orange</material>
-      <mu1>0.5</mu1>
-      <mu2>0.5</mu2>
   </gazebo>
   <gazebo reference="${prefix}link_4">
       <material>Gazebo/Grey</material>
-      <mu1>0.5</mu1>
-      <mu2>0.5</mu2>
   </gazebo>
   <gazebo reference="${prefix}link_5">
       <material>Gazebo/Green</material>
-      <mu1>0.5</mu1>
-      <mu2>0.5</mu2>
   </gazebo>
   <gazebo reference="${prefix}link_6">
       <material>Gazebo/Blue</material>
-      <mu1>0.5</mu1>
-      <mu2>0.5</mu2>
   </gazebo>
   <gazebo reference="${prefix}link_7">
       <material>Gazebo/Yellow</material>
-      <mu1>0.5</mu1>
-      <mu2>0.5</mu2>
   </gazebo>
   <gazebo reference="${prefix}pan_link">
       <material>Gazebo/Black</material>
-      <mu1>0.5</mu1>
-      <mu2>0.5</mu2>
   </gazebo>
   <gazebo reference="${prefix}xiao_arm1_link">
       <material>Gazebo/White</material>
-      <mu1>0.5</mu1>
-      <mu2>0.5</mu2>
   </gazebo>
   <gazebo reference="${prefix}xiao_arm2_link">
       <material>Gazebo/Green</material>
-      <mu1>0.5</mu1>
-      <mu2>0.5</mu2>
   </gazebo>
   <gazebo reference="${prefix}xiangji_link">
       <material>Gazebo/Orange</material>
-      <mu1>0.5</mu1>
-      <mu2>0.5</mu2>
   </gazebo>
   <!--ros control plugin-->
@@ -70,5 +44,4 @@
     <plugin name="gazebo_ros_control" filename="libgazebo_ros_control.so">
       <robotNamespace>/iiwa</robotNamespace>
-      <robotParam>/iiwa/robot_description</robotParam>
       <robotSimType>gazebo_ros_control/DefaultRobotHWSim</robotSimType>
       <!--legacyModeNS>true</legacyModeNS-->

File: urdf/iiwa_agv.urdf.xacro (robot description, xacro)
@@ -2,7 +2,9 @@
 <robot name="iiwa_agv" xmlns:xacro="http://wiki.ros.org/xacro">
   <!-- some xacro properties-->
-  <xacro:property name="pi" value="3.1415926535897931" />
+  <xacro:property name="PI" value="3.1415926535897931" />
   <xacro:property name="prefix" value="" />
   <xacro:property name="agv_mass" value="50.0" />
+  <xacro:property name="xiao_arm_offset_x" value="0.15" />
+  <xacro:property name="xiao_arm_offset_y" value="0.5" />
   <!-- include the xacro files-->
   <xacro:include filename="$(find iiwa_agv)/urdf/iiwa_agv.transmission.xacro"/>
@@ -26,5 +28,5 @@
     </inertial>
     <visual>
-      <origin xyz="0 0 0" rpy="1.570796 0 0" />
+      <origin xyz="0 0 0" rpy="${PI/2.0} 0 0" />
       <geometry>
         <mesh filename="package://gazebo_example/meshes/che.STL" />
@@ -33,5 +35,5 @@
     </visual>
     <collision>
-      <origin xyz="0 0 0" rpy="1.570796 0 0" />
+      <origin xyz="0 0 0" rpy="${PI/2.0} 0 0" />
       <geometry>
         <mesh filename="package://iiwa_agv/meshes/che.STL" />
@@ -186,4 +188,5 @@
   <link name="${prefix}pan_link">
     <visual>
+      <origin xyz="0 0 0" rpy="${PI/2.0} 0 0" />
       <geometry>
         <mesh filename="package://iiwa_agv/meshes/pan.STL"/>
@@ -192,14 +195,16 @@
     </visual>
     <collision>
+      <origin xyz="0 0 0" rpy="${PI/2.0} 0 0" />
       <geometry>
         <mesh filename="package://iiwa_agv/meshes/pan.STL"/>
       </geometry>
     </collision>
-    <xacro:cylinder_inertial radius="0.05" length="0.01" mass="0.01">
-      <origin xyz="0.0 0.0 0.0" rpy="0 0 0" />
+    <xacro:cylinder_inertial radius="0.25" length="0.1" mass="0.01">
+      <origin xyz="0.0 0.0 0.0" rpy="${PI/2.0} 0 0" />
     </xacro:cylinder_inertial>
   </link>
   <link name="${prefix}xiao_arm1_link">
     <visual>
+      <origin xyz="0 ${xiao_arm_offset_y} 0.02" rpy="${PI/2.0} 0 0" />
       <geometry>
         <mesh filename="package://iiwa_agv/meshes/xiao_arm.STL"/>
@@ -208,14 +213,16 @@
     </visual>
     <collision>
-      <geometry>
-        <mesh filename="package://iiwa_agv/meshes/xiao_arm.STL"/>
-      </geometry>
-    </collision>
-    <xacro:cylinder_inertial radius="0.05" length="0.01" mass="0.01">
-      <origin xyz="0.0 0.0 0.0" rpy="0 0 0" />
+      <origin xyz="0 ${xiao_arm_offset_y} 0.02" rpy="${PI/2.0} 0 0" />
+      <geometry>
+        <mesh filename="package://iiwa_agv/meshes/xiao_arm.STL"/>
+      </geometry>
+    </collision>
+    <xacro:cylinder_inertial radius="0.01" length="0.05" mass="0.01">
+      <origin xyz="0.1 0.0 0.25" rpy="0 0 0" />
     </xacro:cylinder_inertial>
   </link>
   <link name="${prefix}xiao_arm2_link">
     <visual>
+      <origin xyz="${-xiao_arm_offset_x} ${xiao_arm_offset_y} 0.02" rpy="${PI/2.0} 0 0" />
       <geometry>
         <mesh filename="package://iiwa_agv/meshes/xiao_arm.STL"/>
@@ -224,14 +231,16 @@
     </visual>
     <collision>
-      <geometry>
-        <mesh filename="package://iiwa_agv/meshes/xiao_arm.STL"/>
-      </geometry>
-    </collision>
-    <xacro:cylinder_inertial radius="0.05" length="0.01" mass="0.01">
-      <origin xyz="0.0 0.0 0.0" rpy="0 0 0" />
+      <origin xyz="${-xiao_arm_offset_x} ${xiao_arm_offset_y} 0.02" rpy="${PI/2.0} 0 0" />
+      <geometry>
+        <mesh filename="package://iiwa_agv/meshes/xiao_arm.STL"/>
+      </geometry>
+    </collision>
+    <xacro:cylinder_inertial radius="0.01" length="0.05" mass="0.01">
+      <origin xyz="-0.1 0.0 0.25" rpy="0 0 0" />
     </xacro:cylinder_inertial>
   </link>
   <link name="${prefix}xiangji_link">
     <visual>
+      <origin xyz="0.0 0.0 0.1" rpy="0 0 0" />
       <geometry>
         <mesh filename="package://iiwa_agv/meshes/xiangji.STL"/>
@@ -240,9 +249,10 @@
     </visual>
     <collision>
-      <geometry>
-        <mesh filename="package://iiwa_agv/meshes/xiao_arm.STL"/>
-      </geometry>
-    </collision>
-    <xacro:cylinder_inertial radius="0.05" length="0.01" mass="0.01">
+      <origin xyz="0.0 0.0 0.07" rpy="0 0 0" />
+      <geometry>
+        <mesh filename="package://iiwa_agv/meshes/xiao_arm.STL"/>
+      </geometry>
+    </collision>
+    <xacro:cylinder_inertial radius="0.01" length="0.05" mass="0.01">
       <origin xyz="0.0 0.0 0.0" rpy="0 0 0" />
     </xacro:cylinder_inertial>
@@ -313,28 +323,20 @@
     <parent link="${prefix}link_7" />
     <child link = "${prefix}pan_link" />
-    <origin xyz="0.0 0.0 0.12" rpy="1.5708 0.0 0.0" />
-    <axis xyz="0 1 0" />
-    <dynamics damping="0.0" friction="0.0"/>
+    <origin xyz="0.0 0.0 0.126" rpy="0.0 0.0 0.0" />
   </joint>
   <joint name="${prefix}pan_to_xiao_arm1_joint" type="fixed">
     <parent link="${prefix}pan_link" />
     <child link = "${prefix}xiao_arm1_link" />
-    <origin xyz="0.0 0.0 -0.47" rpy="0.0 0.0 0.0" />
-    <axis xyz="0 1 0" />
-    <dynamics damping="0.0" friction="0.0"/>
+    <origin xyz="0.0 0.0 0.0" rpy="0.0 0.0 0.0" />
   </joint>
   <joint name="${prefix}pan_to_xiao_arm2_joint" type="fixed">
     <parent link="${prefix}pan_link" />
     <child link = "${prefix}xiao_arm2_link" />
-    <origin xyz="-0.15 0.0 -0.47" rpy="0.0 0.0 0.0" />
-    <axis xyz="0 1 0" />
-    <dynamics damping="0.0" friction="0.0"/>
+    <origin xyz="0.0 0.0 0.0" rpy="0.0 0.0 0.0" />
   </joint>
   <joint name="${prefix}pan_to_xiangji_joint" type="fixed">
     <parent link="${prefix}pan_link" />
     <child link = "${prefix}xiangji_link" />
-    <origin xyz="0.0 0.065 -0.1" rpy="-1.570796 0.0 0.0" />
-    <axis xyz="0 1 0" />
-    <dynamics damping="0.0" friction="0.0"/>
+    <origin xyz="0.0 0.0 0.0" rpy="0.0 0.0 0.0" />
   </joint>
   <!-- end of joint list -->

Commit message: chg support axis

File: urdf/iiwa_agv.gazebo.xacro (robot description, xacro)
@@ -49,5 +49,5 @@
   </gazebo>
   <!--move_base plugin -->
-  <gazebo>
+  <!--gazebo>
     <plugin name="base_controller" filename="libgazebo_ros_planar_move.so">
       <commandTopic>/base/cmd_vel</commandTopic>
@@ -57,4 +57,4 @@
       <robotBaseFrame>agv_link</robotBaseFrame>
     </plugin>
-  </gazebo>
+  </gazebo-->
 </robot>

File: urdf/iiwa_agv.urdf.xacro (robot description, xacro)
@@ -55,5 +55,5 @@
         <parent link="${prefix}virtual_base"/>
         <child link="${prefix}virtual_x"/>
-        <axis xyz="0.0 1.0 0.0"/>
+        <axis xyz="1.0 0.0 0.0"/>
         <limit lower="-5.0" upper="5.0" effort="50.0" velocity="2.0"/>
     </joint>
@@ -62,5 +62,5 @@
         <parent link="${prefix}virtual_x"/>
         <child link="${prefix}virtual_y"/>
-        <axis xyz="-1.0 0.0 0.0"/>
+        <axis xyz="0.0 1.0 0.0"/>
         <limit lower="-5.0" upper="5.0" effort="50.0" velocity="2.0"/>
     </joint>
