Commit message: add excutor & chg pid

File: urdf/iiwa_agv.urdf.xacro (robot description, xacro)
@@ -28,14 +28,14 @@
     </inertial>
     <visual>
-      <origin xyz="0 0 0" rpy="${PI/2.0} 0 0" />
-      <geometry>
-        <mesh filename="package://gazebo_example/meshes/che.STL" />
+      <origin xyz="0 0 0" rpy="0 0 0" />
+      <geometry>
+        <box size="1 0.5 0.36"/>
       </geometry>
       <material name="blue"/>
     </visual>
     <collision>
-      <origin xyz="0 0 0" rpy="${PI/2.0} 0 0" />
-      <geometry>
-        <mesh filename="package://iiwa_agv/meshes/che.STL" />
+      <origin xyz="0 0 0" rpy="0 0 0" />
+      <geometry>
+        <box size="1 0.5 0.36"/>
       </geometry>
     </collision>
@@ -261,5 +261,5 @@
   <!-- joint list -->
   <joint name="${prefix}agv_to_base_joint" type="fixed">
-    <origin xyz="0 0 0.23" rpy="0 0 0" />
+    <origin xyz="0 0 0.18" rpy="0 0 0" />
     <parent link="${prefix}agv_link" />
     <child link="${prefix}base_link" />

Commit message: add support urdf

File: urdf/iiwa_agv.urdf.xacro (robot description, xacro)
@@ -7,8 +7,12 @@
   <xacro:property name="xiao_arm_offset_x" value="0.15" />
   <xacro:property name="xiao_arm_offset_y" value="0.5" />
+  <xacro:property name="agv_height" value="0.36" />
+  <xacro:property name="little_mass" value="0.01"/>
+  <xacro:property name="little_width" value="0.001"/>
   <!-- include the xacro files-->
   <xacro:include filename="$(find iiwa_agv)/urdf/iiwa_agv.transmission.xacro"/>
   <xacro:include filename="$(find iiwa_agv)/urdf/iiwa_agv.gazebo.xacro"/>
   <xacro:include filename="$(find iiwa_agv)/urdf/materials.xacro"/>
+  <xacro:include filename="$(find iiwa_agv)/urdf/support.urdf.xacro"/>
   <!-- some xacro macros-->
   <xacro:macro name="cylinder_inertial" params="radius length mass *origin">
@@ -30,5 +34,5 @@
       <origin xyz="0 0 0" rpy="0 0 0" />
       <geometry>
-        <box size="1 0.5 0.36"/>
+        <box size="1 0.5 ${agv_height}"/>
       </geometry>
       <material name="blue"/>

Commit message: add initial xy offset in urdf

File: urdf/iiwa_agv.urdf.xacro (robot description, xacro)
@@ -7,4 +7,6 @@
   <xacro:property name="xiao_arm_offset_x" value="0.15" />
   <xacro:property name="xiao_arm_offset_y" value="0.5" />
+  <xacro:property name="initial_x" value="0.0" />
+  <xacro:property name="initial_y" value="1.5" />
   <!-- include the xacro files-->
   <xacro:include filename="$(find iiwa_agv)/urdf/iiwa_agv.transmission.xacro"/>
@@ -22,4 +24,5 @@
   </xacro:macro>
   <!-- link list -->
+    <link name="world"/>
     <link name="${prefix}virtual_base">
         <inertial>
@@ -43,4 +46,9 @@
         </inertial>
     </link>
+    <joint name="world_base" type="fixed">
+      <origin xyz="${initial_x} ${initial_y} 0.0" rpy="0.0 0.0 0.0"/>
+      <parent link="world"/>
+      <child link="${prefix}virtual_base"/>
+    </joint>
     <joint name="${prefix}base_x" type="prismatic">
         <origin xyz="0.0 0.0 0.18" rpy="0.0 0.0 0.0"/>

Commit message: neutralize initial xy offset in read

File: urdf/iiwa_agv.urdf.xacro (robot description, xacro)
@@ -65,10 +65,10 @@
         <limit lower="-5.0" upper="5.0" effort="50.0" velocity="2.0"/>
     </joint>
-    <joint name="${prefix}y_car" type="revolute">
+    <joint name="${prefix}y_car" type="continuous">
         <origin xyz="0.0 0.0 0.0" rpy="0.0 0.0 0.0"/>
         <parent link="${prefix}virtual_y"/>
         <child link="${prefix}agv_link"/>
         <axis xyz="0.0 0.0 1.0"/>
-        <limit lower="${-PI}" upper="${PI}" effort="50.0" velocity="2.0"/>
+        <limit effort="50.0" velocity="2.0"/>
     </joint>
   <link name="${prefix}agv_link">

Commit message: update he data & turn iiwa-agv by pi

File: urdf/iiwa_agv.urdf.xacro (robot description, xacro)
@@ -311,5 +311,5 @@
   <!-- joint list -->
   <joint name="${prefix}agv_to_base_joint" type="fixed">
-    <origin xyz="0 0 0.18" rpy="0 0 ${PI}" />
+    <origin xyz="0 0 0.18" rpy="0 0 0" />
     <parent link="${prefix}agv_link" />
     <child link="${prefix}base_link" />

Commit message: chg car stl

File: urdf/iiwa_agv.urdf.xacro (robot description, xacro)
@@ -78,16 +78,16 @@
     </inertial>
     <visual>
-      <origin xyz="0 0 0" rpy="0 0 0" />
-      <geometry>
-        <box size="1 0.5 0.36"/>
-      </geometry>
-      <material name="blue"/>
-    </visual>
-    <collision>
-      <origin xyz="0 0 0" rpy="0 0 0" />
-      <geometry>
-        <box size="1 0.5 0.36"/>
-      </geometry>
-    </collision>
+            <geometry>
+                <mesh filename="package://parallel_car/meshes/car.STL" />
+     	    </geometry>
+            <material name="green"/>
+            <origin rpy="${PI/2.0} 0.0 0.0" xyz="0 0 -0.12"/>
+        </visual>
+        <collision>
+            <geometry>
+                <mesh filename="package://parallel_car/meshes/car.STL" />
+     	    </geometry>
+            <origin rpy="${PI/2.0} 0.0 0.0" xyz="0 0 -0.12"/>
+        </collision>
   </link>
   <link name="${prefix}base_link">
